File: USB2GPIO.kicad_sch (KiCad schematic)
At the start: 11 parts, among them J9 Conn_01x04

Commit message: PCB drawn
Parts:
- C28, C29: value (none) -> 100n; footprint (none) -> Capacitor_SMD:C_0603_1608Metric
- D10, D11, D12: value (none) -> BV05C; footprint (none) -> Diode_SMD:D_SOD-323
- D9: value (none) -> LED; footprint (none) -> LED_SMD:LED_0603_1608Metric
- J1: renamed from J?; footprint (none) -> Connector_JST:JST_EH_S4B-EH_1x04_P2.50mm_Horizontal
- J7, J8: value (none) -> Conn_01x03; footprint (none) -> Connector_JST:JST_GH_SM03B-GHS-TB_1x03-1MP_P1.25mm_Horizontal
- J9: footprint (none) -> Connector_JST:JST_GH_SM04B-GHS-TB_1x04-1MP_P1.25mm_Horizontal
- R14: value (none) -> 1K; footprint (none) -> Resistor_SMD:R_0603_1608Metric
